Commit message: Implemented force estimator and added dynamics functions to KDL interface

File: climb_main/test/resources/test_robot.urdf (robot description, URDF)
Before this commit: robot test_robot, 10 links, 9 joints
Links:
- link body: mass None -> 2
- link left_foot: mass None -> 1
- link right_foot: mass None -> 1
