Commit message: Added Gazebo simulation

File: robot_description/loris_description/urdf/loris.urdf.xacro (robot description, xacro)
@@ -131,6 +131,6 @@
       lower="-1.22173"
       upper="1.22173"
-      effort="0"
-      velocity="0" />
+      effort="4.1"
+      velocity="4.8" />
   </joint>
   <link
@@ -187,6 +187,6 @@
       lower="-1.2217"
       upper="1.5708"
-      effort="0"
-      velocity="0" />
+      effort="4.1"
+      velocity="4.8" />
   </joint>
   <link
@@ -243,6 +243,6 @@
       lower="-1.5708"
       upper="1.0472"
-      effort="0"
-      velocity="0" />
+      effort="4.1"
+      velocity="4.8" />
   </joint>
   <link
@@ -350,6 +350,6 @@
       lower="-1.2217"
       upper="1.2217"
-      effort="0"
-      velocity="0" />
+      effort="4.1"
+      velocity="4.8" />
   </joint>
   <link
@@ -406,6 +406,6 @@
       lower="-1.2217"
       upper="1.570796"
-      effort="0"
-      velocity="0" />
+      effort="4.1"
+      velocity="4.8" />
   </joint>
   <link
@@ -462,6 +462,6 @@
       lower="-1.5708"
       upper="1.047198"
-      effort="0"
-      velocity="0" />
+      effort="4.1"
+      velocity="4.8" />
   </joint>
   <link
@@ -569,6 +569,6 @@
       lower="-1.047198"
       upper="1.047198"
-      effort="0"
-      velocity="0" />
+      effort="4.1"
+      velocity="4.8" />
   </joint>
   <link
@@ -625,6 +625,6 @@
       lower="-1.22173"
       upper="1.22173"
-      effort="0"
-      velocity="0" />
+      effort="4.1"
+      velocity="4.8" />
   </joint>
   <link
@@ -681,6 +681,6 @@
       lower="-1.2217"
       upper="1.570796"
-      effort="0"
-      velocity="0" />
+      effort="4.1"
+      velocity="4.8" />
   </joint>
   <link
@@ -737,6 +737,6 @@
       lower="-1.5708"
       upper="1.047198"
-      effort="0"
-      velocity="0" />
+      effort="4.1"
+      velocity="4.8" />
   </joint>
   <link
@@ -844,6 +844,6 @@
       lower="-1.22173"
       upper="1.22173"
-      effort="0"
-      velocity="0" />
+      effort="4.1"
+      velocity="4.8" />
   </joint>
   <link
@@ -900,6 +900,6 @@
       lower="-1.2217"
       upper="1.570796"
-      effort="0"
-      velocity="0" />
+      effort="4.1"
+      velocity="4.8" />
   </joint>
   <link
@@ -956,6 +956,6 @@
       lower="-1.570796"
       upper="1.047198"
-      effort="0"
-      velocity="0" />
+      effort="4.1"
+      velocity="4.8" />
   </joint>
   <link
@@ -1063,6 +1063,100 @@
       lower="-1.3963"
       upper="1.3963"
-      effort="0"
-      velocity="0" />
-  </joint>
+      effort="4.1"
+      velocity="4.8" />
+  </joint>
+  <ros2_control name="GazeboSystem" type="system">
+    <hardware>
+      <plugin>gz_ros2_control/GazeboSimSystem</plugin>
+    </hardware>
+    <joint name="shoulder_joint_1">
+      <command_interface name="position"/>
+      <state_interface name="position"/>
+      <state_interface name="velocity"/>
+      <state_interface name="effort"/>
+    </joint>
+    <joint name="shoulder_joint_2">
+      <command_interface name="position"/>
+      <state_interface name="position"/>
+      <state_interface name="velocity"/>
+      <state_interface name="effort"/>
+    </joint>
+    <joint name="shoulder_joint_3">
+      <command_interface name="position"/>
+      <state_interface name="position"/>
+      <state_interface name="velocity"/>
+      <state_interface name="effort"/>
+    </joint>
+    <joint name="shoulder_joint_4">
+      <command_interface name="position"/>
+      <state_interface name="position"/>
+      <state_interface name="velocity"/>
+      <state_interface name="effort"/>
+    </joint>
+    <joint name="knee_joint_1">
+      <command_interface name="position"/>
+      <state_interface name="position"/>
+      <state_interface name="velocity"/>
+      <state_interface name="effort"/>
+    </joint>
+    <joint name="knee_joint_2">
+      <command_interface name="position"/>
+      <state_interface name="position"/>
+      <state_interface name="velocity"/>
+      <state_interface name="effort"/>
+    </joint>
+    <joint name="knee_joint_3">
+      <command_interface name="position"/>
+      <state_interface name="position"/>
+      <state_interface name="velocity"/>
+      <state_interface name="effort"/>
+    </joint>
+    <joint name="knee_joint_4">
+      <command_interface name="position"/>
+      <state_interface name="position"/>
+      <state_interface name="velocity"/>
+      <state_interface name="effort"/>
+    </joint>
+    <joint name="wing_joint_1">
+      <command_interface name="position"/>
+      <state_interface name="position"/>
+      <state_interface name="velocity"/>
+      <state_interface name="effort"/>
+    </joint>
+    <joint name="wing_joint_2">
+      <command_interface name="position"/>
+      <state_interface name="position"/>
+      <state_interface name="velocity"/>
+      <state_interface name="effort"/>
+    </joint>
+    <joint name="wing_joint_3">
+      <command_interface name="position"/>
+      <state_interface name="position"/>
+      <state_interface name="velocity"/>
+      <state_interface name="effort"/>
+    </joint>
+    <joint name="wing_joint_4">
+      <command_interface name="position"/>
+      <state_interface name="position"/>
+      <state_interface name="velocity"/>
+      <state_interface name="effort"/>
+    </joint>
+    <joint name="spine_joint">
+      <command_interface name="position"/>
+      <state_interface name="position"/>
+      <state_interface name="velocity"/>
+      <state_interface name="effort"/>
+    </joint>
+    <joint name="tail_joint">
+      <command_interface name="position"/>
+      <state_interface name="position"/>
+      <state_interface name="velocity"/>
+      <state_interface name="effort"/>
+    </joint>
+  </ros2_control>
+  <gazebo>
+    <plugin filename="gz_ros2_control-system" name="gz_ros2_control::GazeboSimROS2ControlPlugin">
+      <parameters>$(find loris_description)/config/gz_params.yaml</parameters>
+    </plugin>
+  </gazebo>
 </robot>

Commit message: Publishing forces from controller node

File: robot_description/loris_description/urdf/loris.urdf.xacro (robot description, xacro)
@@ -293,5 +293,5 @@
       link="lower_limb_1" />
     <child
-      link="gripper_1" />
+      link="wrist_1" />
     <axis
       xyz="0 0 0" />
@@ -512,5 +512,5 @@
       link="lower_limb_2" />
     <child
-      link="gripper_2" />
+      link="wrist_2" />
     <axis
       xyz="0 0 0" />
@@ -787,5 +787,5 @@
       link="lower_limb_3" />
     <child
-      link="gripper_3" />
+      link="wrist_3" />
     <axis
       xyz="0 0 0" />
@@ -1006,7 +1006,27 @@
       link="lower_limb_4" />
     <child
-      link="gripper_4" />
+      link="wrist_4" />
     <axis
       xyz="0 0 0" />
+  </joint>
+  <link name="wrist_1" />
+  <joint name="gripper_joint_1" type="fixed">
+    <parent link="wrist_1"/>
+    <child link="gripper_1"/>
+  </joint>
+  <link name="wrist_2" />
+  <joint name="gripper_joint_2" type="fixed">
+    <parent link="wrist_2"/>
+    <child link="gripper_2"/>
+  </joint>
+  <link name="wrist_3" />
+  <joint name="gripper_joint_3" type="fixed">
+    <parent link="wrist_3"/>
+    <child link="gripper_3"/>
+  </joint>
+  <link name="wrist_4" />
+  <joint name="gripper_joint_4" type="fixed">
+    <parent link="wrist_4"/>
+    <child link="gripper_4"/>
   </joint>
   <link
@@ -1065,4 +1085,15 @@
       effort="4.1"
       velocity="4.8" />
+  </joint>
+  <link name="tail_tip" />
+  <joint name="tail_tip_joint" type="fixed">
+    <parent link="tail"/>
+    <child link="tail_tip"/>
+    <origin xyz="0.35 0 0" rpy="0 1.5708 0"/>
+  </joint>
+  <link name="tail_contact" />
+  <joint name="tail_contact_joint" type="fixed">
+    <parent link="tail_tip"/>
+    <child link="tail_contact"/>
   </joint>
   <ros2_control name="GazeboSystem" type="system">

Commit message: Improved invalid parameter handling

File: robot_description/loris_description/urdf/loris.urdf.xacro (robot description, xacro)
@@ -44,5 +44,5 @@
     <inertial>
       <origin
-        xyz="0.088526 4.9542E-05 0.019968"
+        xyz="0.0811300558392716 -0.000405929819738513 0.00121008339941299"
         rpy="0 0 0" />
       <mass
@@ -523,12 +523,12 @@
         rpy="0 0 0" />
       <mass
-        value="3.13423337298763" />
-      <inertia
-        ixx="0.00626707152969831"
-        ixy="-4.70768643254072E-13"
-        ixz="-3.51127834155193E-08"
-        iyy="0.00809676727966312"
-        iyz="-2.02700054710046E-13"
-        izz="0.0134099994197008" />
+        value="0.87565" />
+      <inertia
+        ixx="0.0014577"
+        ixy="3.0574E-07"
+        ixz="1.0637E-07"
+        iyy="0.0017823"
+        iyz="-1.4776E-07"
+        izz="0.0029263" />
     </inertial>
     <visual>

Commit message: Began Gazebo grasp plugin development

File: robot_description/loris_description/urdf/loris.urdf.xacro (robot description, xacro)
@@ -250,5 +250,5 @@
     <inertial>
       <origin
-        xyz="0.00454536689668263 6.93889390390723E-16 0.000630502612849193"
+        xyz="0.00454536689668263 6.93889390390723E-16 -0.02"
         rpy="0 0 0" />
       <mass
@@ -285,5 +285,5 @@
   </link>
   <joint
-    name="wrist_joint_1"
+    name="wrist_joint_1a"
     type="fixed">
     <origin
@@ -293,5 +293,5 @@
       link="lower_limb_1" />
     <child
-      link="wrist_1" />
+      link="wrist_1a" />
     <axis
       xyz="0 0 0" />
@@ -469,5 +469,5 @@
     <inertial>
       <origin
-        xyz="0.00454536689668164 -1.63757896132211E-15 0.000630502612847555"
+        xyz="0.00454536689668164 -1.63757896132211E-15 -0.02"
         rpy="0 0 0" />
       <mass
@@ -504,5 +504,5 @@
   </link>
   <joint
-    name="wrist_joint_2"
+    name="wrist_joint_2a"
     type="fixed">
     <origin
@@ -512,5 +512,5 @@
       link="lower_limb_2" />
     <child
-      link="wrist_2" />
+      link="wrist_2a" />
     <axis
       xyz="0 0 0" />
@@ -744,5 +744,5 @@
     <inertial>
       <origin
-        xyz="0.00454536689668293 -1.07414077632484E-14 0.000630502612850609"
+        xyz="0.00454536689668293 -1.07414077632484E-14 -0.02"
         rpy="0 0 0" />
       <mass
@@ -779,5 +779,5 @@
   </link>
   <joint
-    name="wrist_joint_3"
+    name="wrist_joint_3a"
     type="fixed">
     <origin
@@ -787,5 +787,5 @@
       link="lower_limb_3" />
     <child
-      link="wrist_3" />
+      link="wrist_3a" />
     <axis
       xyz="0 0 0" />
@@ -963,5 +963,5 @@
     <inertial>
       <origin
-        xyz="0.00454536689667982 1.301736496373E-14 0.000630502612845113"
+        xyz="0.00454536689667982 1.301736496373E-14 -0.02"
         rpy="0 0 0" />
       <mass
@@ -998,5 +998,5 @@
   </link>
   <joint
-    name="wrist_joint_4"
+    name="wrist_joint_4a"
     type="fixed">
     <origin
@@ -1006,27 +1006,127 @@
       link="lower_limb_4" />
     <child
-      link="wrist_4" />
+      link="wrist_4a" />
     <axis
       xyz="0 0 0" />
   </joint>
-  <link name="wrist_1" />
-  <joint name="gripper_joint_1" type="fixed">
-    <parent link="wrist_1"/>
+  <link name="wrist_1a" />
+  <link name="wrist_1b">
+    <inertial>
+      <mass value="1e-3"/>
+      <inertia ixx="1e-5" ixy="0" ixz="0" iyy="1e-5" iyz="0" izz="1e-5" />
+    </inertial>
+  </link>
+  <link name="wrist_1c">
+    <inertial>
+      <mass value="1e-3"/>
+      <inertia ixx="1e-5" ixy="0" ixz="0" iyy="1e-5" iyz="0" izz="1e-5" />
+    </inertial>
+  </link>
+  <joint name="wrist_joint_1b" type="continuous">
+    <parent link="wrist_1a"/>
+    <child link="wrist_1b"/>
+    <axis xyz="1 0 0" />
+  </joint>
+  <joint name="wrist_joint_1c" type="revolute">
+    <parent link="wrist_1b"/>
+    <child link="wrist_1c"/>
+    <axis xyz="0 1 0" />
+    <limit lower="-0.61" upper="0.61" effort="0" velocity="4.8" />
+  </joint>
+  <joint name="gripper_joint_1" type="revolute">
+    <parent link="wrist_1c"/>
     <child link="gripper_1"/>
-  </joint>
-  <link name="wrist_2" />
-  <joint name="gripper_joint_2" type="fixed">
-    <parent link="wrist_2"/>
+    <axis xyz="0 0 1" />
+    <limit lower="-0.61" upper="0.61" effort="0" velocity="4.8" />
+  </joint>
+  <link name="wrist_2a" />
+  <link name="wrist_2b">
+    <inertial>
+      <mass value="1e-3"/>
+      <inertia ixx="1e-5" ixy="0" ixz="0" iyy="1e-5" iyz="0" izz="1e-5" />
+    </inertial>
+  </link>
+  <link name="wrist_2c">
+    <inertial>
+      <mass value="1e-3"/>
+      <inertia ixx="1e-5" ixy="0" ixz="0" iyy="1e-5" iyz="0" izz="1e-5" />
+    </inertial>
+  </link>
+  <joint name="wrist_joint_2b" type="continuous">
+    <parent link="wrist_2a"/>
+    <child link="wrist_2b"/>
+    <axis xyz="1 0 0" />
+  </joint>
+  <joint name="wrist_joint_2c" type="revolute">
+    <parent link="wrist_2b"/>
+    <child link="wrist_2c"/>
+    <axis xyz="0 1 0" />
+    <limit lower="-0.61" upper="0.61" effort="0" velocity="4.8" />
+  </joint>
+  <joint name="gripper_joint_2" type="revolute">
+    <parent link="wrist_2c"/>
     <child link="gripper_2"/>
-  </joint>
-  <link name="wrist_3" />
-  <joint name="gripper_joint_3" type="fixed">
-    <parent link="wrist_3"/>
+    <axis xyz="0 0 1" />
+    <limit lower="-0.61" upper="0.61" effort="0" velocity="4.8" />
+  </joint>
+  <link name="wrist_3a" />
+  <link name="wrist_3b">
+    <inertial>
+      <mass value="1e-3"/>
+      <inertia ixx="1e-5" ixy="0" ixz="0" iyy="1e-5" iyz="0" izz="1e-5" />
+    </inertial>
+  </link>
+  <link name="wrist_3c">
+    <inertial>
+      <mass value="1e-3"/>
+      <inertia ixx="1e-5" ixy="0" ixz="0" iyy="1e-5" iyz="0" izz="1e-5" />
+    </inertial>
+  </link>
+  <joint name="wrist_joint_3b" type="continuous">
+    <parent link="wrist_3a"/>
+    <child link="wrist_3b"/>
+    <axis xyz="1 0 0" />
+  </joint>
+  <joint name="wrist_joint_3c" type="revolute">
+    <parent link="wrist_3b"/>
+    <child link="wrist_3c"/>
+    <axis xyz="0 1 0" />
+    <limit lower="-0.61" upper="0.61" effort="0" velocity="4.8" />
+  </joint>
+  <joint name="gripper_joint_3" type="revolute">
+    <parent link="wrist_3c"/>
     <child link="gripper_3"/>
-  </joint>
-  <link name="wrist_4" />
-  <joint name="gripper_joint_4" type="fixed">
-    <parent link="wrist_4"/>
+    <axis xyz="0 0 1" />
+    <limit lower="-0.61" upper="0.61" effort="0" velocity="4.8" />
+  </joint>
+  <link name="wrist_4a" />
+  <link name="wrist_4b">
+    <inertial>
+      <mass value="1e-3"/>
+      <inertia ixx="1e-5" ixy="0" ixz="0" iyy="1e-5" iyz="0" izz="1e-5" />
+    </inertial>
+  </link>
+  <link name="wrist_4c">
+    <inertial>
+      <mass value="1e-3"/>
+      <inertia ixx="1e-5" ixy="0" ixz="0" iyy="1e-5" iyz="0" izz="1e-5" />
+    </inertial>
+  </link>
+  <joint name="wrist_joint_4b" type="continuous">
+    <parent link="wrist_4a"/>
+    <child link="wrist_4b"/>
+    <axis xyz="1 0 0" />
+  </joint>
+  <joint name="wrist_joint_4c" type="revolute">
+    <parent link="wrist_4b"/>
+    <child link="wrist_4c"/>
+    <axis xyz="0 1 0" />
+    <limit lower="-0.61" upper="0.61" effort="0" velocity="4.8" />
+  </joint>
+  <joint name="gripper_joint_4" type="revolute">
+    <parent link="wrist_4c"/>
     <child link="gripper_4"/>
+    <axis xyz="0 0 1" />
+    <limit lower="-0.61" upper="0.61" effort="0" velocity="4.8" />
   </joint>
   <link
@@ -1186,4 +1286,18 @@
     </joint>
   </ros2_control>
+  <gazebo reference="gripper_joint_1">
+    <preserveFixedJoint>true</preserveFixedJoint>
+    <sensor name="force_torque_sensor" type="force_torque">
+      <pose>0 0 0 0 0 0</pose>
+      <update_rate>100</update_rate>
+      <always_on>true</always_on>
+      <visualize>true</visualize>
+      <topic>force_torque</topic>
+      <force_torque>
+        <frame>child</frame>
+        <measure_direction>child_to_parent</measure_direction>
+      </force_torque>
+    </sensor>
+  </gazebo>
   <gazebo>
     <plugin filename="gz_ros2_control-system" name="gz_ros2_control::GazeboSimROS2ControlPlugin">
