Commit message: Simplified LORIS description with xacro

File: robot_description/loris_description/urdf/loris.urdf.xacro (robot description, xacro)
@@ -1,38 +1,90 @@
 <?xml version="1.0" encoding="utf-8"?>
-<!-- This URDF was automatically created by SolidWorks to URDF Exporter! Originally created by Stephen Brawner (brawner@gmail.com)
-     Commit Version: 1.6.0-4-g7f85cfe  Build Version: 1.6.7995.38578
-     For more information, please see http://wiki.ros.org/sw_urdf_exporter -->
-<robot
-  name="loris">
-  <material
-    name="body_mat">
-    <color
-      rgba="1 1 1 1" />
-  </material>
-  <material
-    name="shoulder_mat">
-    <color
-      rgba="0.25098 0.25098 0.25098 1" />
-  </material>
-  <material
-    name="upper_mat">
-    <color
-      rgba="0.752941176470588 0.752941176470588 0.752941176470588 1" />
-  </material>
-  <material
-    name="lower_mat">
-    <color
-      rgba="0.752941176470588 0.752941176470588 0.752941176470588 1" />
-  </material>
-  <material
-    name="gripper_mat">
-    <color
-      rgba="0.250980392156863 0.250980392156863 0.250980392156863 1" />
-  </material>
-  <material
-    name="tail_mat">
-    <color
-      rgba="0.25098 0.25098 0.25098 1" />
-  </material>
+<!--
+  MIT License
+  Copyright (c) 2024 Paul Nadan, Robomechanics Lab, Carnegie Mellon University
+  Permission is hereby granted, free of charge, to any person obtaining a copy
+  of this software and associated documentation files (the "Software"), to deal
+  in the Software without restriction, including without limitation the rights
+  to use, copy, modify, merge, publish, distribute, sublicense, and/or sell
+  copies of the Software, and to permit persons to whom the Software is
+  furnished to do so, subject to the following conditions:
+  The above copyright notice and this permission notice shall be included in
+  all copies or substantial portions of the Software.
+  THE SOFTWARE IS PROVIDED "AS IS", WITHOUT WARRANTY OF ANY KIND, EXPRESS OR
+  IMPLIED, INCLUDING BUT NOT LIMITED TO THE WARRANTIES OF MERCHANTABILITY,
+  FITNESS FOR A PARTICULAR PURPOSE AND NONINFRINGEMENT. IN NO EVENT SHALL
+  THE AUTHORS OR COPYRIGHT HOLDERS BE LIABLE FOR ANY CLAIM, DAMAGES OR OTHER
+  LIABILITY, WHETHER IN AN ACTION OF CONTRACT, TORT OR OTHERWISE, ARISING FROM,
+  OUT OF OR IN CONNECTION WITH THE SOFTWARE OR THE USE OR OTHER DEALINGS IN
+  THE SOFTWARE.
+-->
+<robot xmlns:xacro="http://www.ros.org/wiki/xacro" name="loris">
+  <!-- Represent wrist as 1 floating joint instead of 3 passive joints -->
+  <xacro:arg name="floating_wrist" default="false" />
+  <xacro:property name="floating_wrist" value="$(arg floating_wrist)" />
+  <!-- Camera mounting height (m from body origin to pitch axis) -->
+  <xacro:arg name="camera_height" default="0.181" />
+  <xacro:property name="camera_height" value="$(arg camera_height)" />
+  <!-- Camera mounting pitch (deg downward from horizontal) -->
+  <xacro:arg name="camera_pitch" default="25" />
+  <xacro:property name="camera_pitch" value="$(arg camera_pitch)" />
+  <!-- Gripper angle offsets (deg outward from centerline) -->
+  <xacro:arg name="gripper_offset" default="45" />
+  <xacro:arg name="gripper_offset_1" default="$(arg gripper_offset)" />
+  <xacro:arg name="gripper_offset_2" default="$(arg gripper_offset)" />
+  <xacro:arg name="gripper_offset_3" default="$(arg gripper_offset)" />
+  <xacro:arg name="gripper_offset_4" default="$(arg gripper_offset)" />
+  <xacro:property name="gripper_offset_1" value="$(arg gripper_offset_1)" />
+  <xacro:property name="gripper_offset_2" value="$(arg gripper_offset_2)" />
+  <xacro:property name="gripper_offset_3" value="$(arg gripper_offset_3)" />
+  <xacro:property name="gripper_offset_4" value="$(arg gripper_offset_4)" />
+  <!-- Actuator Limits (Nm and rad/s) -->
+  <xacro:arg name="effort" default="4.1" />
+  <xacro:arg name="velocity" default="4.8" />
+  <xacro:property name="effort" value="$(arg effort)" />
+  <xacro:property name="velocity" value="$(arg velocity)" />
+  <!-- Mesh directories -->
+  <xacro:property name="visual" value="package://loris_description/meshes" />
+  <xacro:property name="collision" value="package://loris_description/meshes" />
+  <!-- Material Properties -->
+  <material name="body_material">
+    <color rgba="1 1 1 1" />
+  </material>
+  <material name="shoulder_material">
+    <color rgba="0.25 0.25 0.25 1" />
+  </material>
+  <material name="upper_limb_material">
+    <color rgba="0.75 0.75 0.75 1" />
+  </material>
+  <material name="lower_limb_material">
+    <color rgba="0.75 0.75 0.75 1" />
+  </material>
+  <material name="gripper_material">
+    <color rgba="0.25 0.25 0.25 1" />
+  </material>
+  <material name="tail_material">
+    <color rgba="0.25 0.25 0.25 1" />
+  </material>
+  <material name="mast_material">
+    <color rgba="0.25 0.25 0.25 1" />
+  </material>
+  <material name="camera_material">
+    <color rgba="1 1 1 1" />
+  </material>
+  <!-- Unit Conversion -->
+  <xacro:property name="deg" value="${pi/180}" />
+  <!-- Normalized Inertia Macro -->
+  <xacro:macro name="inertial"
+    params="mass:=0 ixx:=0 ixy:=0 ixz:=0 iyy:=0 iyz:=0 izz:=0">
+    <mass value="${mass}" />
+    <inertia
+      ixx="${mass * ixx}"
+      ixy="${mass * ixy}"
+      ixz="${mass * ixz}"
+      iyy="${mass * iyy}"
+      iyz="${mass * iyz}"
+      izz="${mass * izz}" />
+  </xacro:macro>
+  <!-- Root frame -->
   <link name="root" />
   <joint name="root_joint" type="fixed">
@@ -40,1049 +92,76 @@
     <child link="body_front" />
   </joint>
-  <link
-    name="body_front">
-    <inertial>
-      <origin
-        xyz="0.0811300558392716 -0.000405929819738513 0.00121008339941299"
-        rpy="0 0 0" />
-      <mass
-        value="0.87565" />
-      <inertia
-        ixx="0.0014577"
-        ixy="3.0574E-07"
-        ixz="1.0637E-07"
-        iyy="0.0017823"
-        iyz="-1.4776E-07"
-        izz="0.0029263" />
-    </inertial>
-    <visual>
-      <origin
-        xyz="0 0 0"
-        rpy="0 0 0" />
-      <geometry>
-        <mesh
-          filename="package://loris_description/meshes/body_front.STL" />
-      </geometry>
-      <material
-        name="body_mat">
-      </material>
-    </visual>
-    <collision>
-      <origin
-        xyz="0 0 0"
-        rpy="0 0 0" />
-      <geometry>
-        <mesh
-          filename="package://loris_description/meshes/body_front.STL" />
-      </geometry>
-    </collision>
-  </link>
-  <link
-    name="shoulder_1">
-    <inertial>
-      <origin
-        xyz="0.015026 0.00033378 5.8541E-05"
-        rpy="0 0 0" />
-      <mass
-        value="0.10342" />
-      <inertia
-        ixx="2.1451E-05"
-        ixy="-4.1299E-07"
-        ixz="3.4401E-08"
-        iyy="2.5017E-05"
-        iyz="1.9009E-08"
-        izz="2.8896E-05" />
-    </inertial>
-    <visual>
-      <origin
-        xyz="0 0 0"
-        rpy="0 0 0" />
-      <geometry>
-        <mesh
-          filename="package://loris_description/meshes/shoulder_1.STL" />
-      </geometry>
-      <material
-        name="shoulder_mat">
-      </material>
-    </visual>
-    <collision>
-      <origin
-        xyz="0 0 0"
-        rpy="0 0 0" />
-      <geometry>
-        <mesh
-          filename="package://loris_description/meshes/shoulder_1.STL" />
-      </geometry>
-    </collision>
-  </link>
-  <joint
-    name="shoulder_joint_1"
-    type="revolute">
-    <origin
-      xyz="0.14145 0.08175 -0.0003"
-      rpy="0 0 1.5708" />
-    <parent
-      link="body_front" />
-    <child
-      link="shoulder_1" />
-    <axis
-      xyz="0 0 -1" />
-    <limit
-      lower="-1.22173"
-      upper="1.22173"
-      effort="4.1"
-      velocity="4.8" />
-  </joint>
-  <link
-    name="upper_limb_1">
-    <inertial>
-      <origin
-        xyz="0.0945138162071381 -0.00219435785796701 -0.00808171492908145"
-        rpy="0 0 0" />
-      <mass
-        value="0.122852357543703" />
-      <inertia
-        ixx="3.54345460928741E-05"
-        ixy="-6.91676719337593E-07"
-        ixz="7.99818931512339E-07"
-        iyy="3.51134789983964E-05"
-        iyz="-2.29657896991753E-12"
-        izz="3.44677592214051E-05" />
-    </inertial>
-    <visual>
-      <origin
-        xyz="0 0 0"
-        rpy="0 0 0" />
-      <geometry>
-        <mesh
-          filename="package://loris_description/meshes/upper_limb_1.STL" />
-      </geometry>
-      <material
-        name="upper_mat">
-      </material>
-    </visual>
-    <collision>
-      <origin
-        xyz="0 0 0"
-        rpy="0 0 0" />
-      <geometry>
-        <mesh
-          filename="package://loris_description/meshes/upper_limb_1.STL" />
-      </geometry>
-    </collision>
-  </link>
-  <joint
-    name="wing_joint_1"
-    type="revolute">
-    <origin
-      xyz="0.02973 0 0"
-      rpy="0 0 0" />
-    <parent
-      link="shoulder_1" />
-    <child
-      link="upper_limb_1" />
-    <axis
-      xyz="0 1 0" />
-    <limit
-      lower="-1.2217"
-      upper="1.5708"
-      effort="4.1"
-      velocity="4.8" />
-  </joint>
-  <link
-    name="lower_limb_1">
-    <inertial>
-      <origin
-        xyz="0.0385688856224721 -0.0046889638702359 -0.00426946293309724"
-        rpy="0 0 0" />
-      <mass
-        value="0.0346530871970472" />
-      <inertia
-        ixx="7.71046451441355E-06"
-        ixy="-3.0991220361643E-07"
-        ixz="3.24361698315945E-06"
-        iyy="1.12808018413156E-05"
-        iyz="-4.85311495827955E-12"
-        izz="1.2230867218234E-05" />
-    </inertial>
-    <visual>
-      <origin
-        xyz="0 0 0"
-        rpy="0 0 0" />
-      <geometry>
-        <mesh
-          filename="package://loris_description/meshes/lower_limb_1.STL" />
-      </geometry>
-      <material
-        name="lower_mat">
-      </material>
-    </visual>
-    <collision>
-      <origin
-        xyz="0 0 0"
-        rpy="0 0 0" />
-      <geometry>
-        <mesh
-          filename="package://loris_description/meshes/lower_limb_1.STL" />
-      </geometry>
-    </collision>
-  </link>
-  <joint
-    name="knee_joint_1"
-    type="revolute">
-    <origin
-      xyz="0.11125 0 -0.02275"
-      rpy="0 1.5708 0" />
-    <parent
-      link="upper_limb_1" />
-    <child
-      link="lower_limb_1" />
-    <axis
-      xyz="0 1 0" />
-    <limit
-      lower="-1.5708"
-      upper="1.0472"
-      effort="4.1"
-      velocity="4.8" />
-  </joint>
-  <link
-    name="gripper_1">
-    <inertial>
-      <origin
-        xyz="0.00454536689668263 6.93889390390723E-16 0.000630502612849193"
-        rpy="0 0 0" />
-      <mass
-        value="0.062469295997667" />
-      <inertia
-        ixx="4.42421322057347E-05"
-        ixy="3.61359625915917E-20"
-        ixz="-8.22176735773703E-07"
-        iyy="1.36212602544054E-05"
-        iyz="9.93950717413035E-19"
-        izz="3.31611786775593E-05" />
-    </inertial>
-    <visual>
-      <origin
-        xyz="0 0 0"
-        rpy="0 0 0" />
-      <geometry>
-        <mesh
-          filename="package://loris_description/meshes/gripper_1.STL" />
-      </geometry>
-      <material
-        name="gripper_mat">
-      </material>
-    </visual>
-    <collision>
-      <origin
-        xyz="0 0 0"
-        rpy="0 0 0" />
-      <geometry>
-        <mesh
-          filename="package://loris_description/meshes/gripper_1.STL" />
-      </geometry>
-    </collision>
-  </link>
-  <joint
-    name="wrist_joint_1"
-    type="fixed">
-    <origin
-      xyz="0.08595 -0.004 -0.02756"
-      rpy="0 0.5236 0" />
-    <parent
-      link="lower_limb_1" />
-    <child
-      link="wrist_1" />
-    <axis
-      xyz="0 0 0" />
-  </joint>
-  <link
-    name="shoulder_2">
-    <inertial>
-      <origin
-        xyz="0.0150259998235379 -0.000333783259922532 5.85409408931406E-05"
-        rpy="0 0 0" />
-      <mass
-        value="0.103423862682087" />
-      <inertia
-        ixx="2.14513424849859E-05"
-        ixy="4.129850457377E-07"
-        ixz="3.44007049222985E-08"
-        iyy="2.5016622013786E-05"
-        iyz="-1.90087151924638E-08"
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
Commit message: RealSense SLAM integration

File: robot_description/loris_description/urdf/loris.urdf.xacro (robot description, xacro)
@@ -24,5 +24,5 @@
   <xacro:property name="floating_wrist" value="$(arg floating_wrist)" />
   <!-- Camera mounting height (m from body origin to pitch axis) -->
-  <xacro:arg name="camera_height" default="0.181" />
+  <xacro:arg name="camera_height" default="0.28" />
   <xacro:property name="camera_height" value="$(arg camera_height)" />
   <!-- Camera mounting pitch (deg downward from horizontal) -->
@@ -196,7 +196,7 @@
   </link>
   <joint name="mast_joint" type="fixed">
-    <origin xyz="0.0247 0 0" />
-    <parent link="body_front" />
-    <child link="mast" />
+    <origin xyz="-0.0247 0 0" />
+    <parent link="mast" />
+    <child link="root" />
   </joint>
   <link name="camera_mount">
@@ -220,7 +220,7 @@
   <joint
     name="camera_mast_joint" type="fixed">
-    <origin xyz="0 0 ${camera_height}" />
-    <parent link="mast" />
-    <child link="camera_mount" />
+    <origin xyz="0 0 ${-camera_height}" />
+    <parent link="camera_mount" />
+    <child link="mast" />
   </joint>
   <link
@@ -244,13 +244,13 @@
   </link>
   <joint name="camera_pitch_joint" type="fixed">
-    <origin xyz="0.0120 0 0" rpy="0 ${camera_pitch * deg} 0" />
-    <parent link="camera_mount" />
-    <child link="camera" />
+    <origin xyz="-0.0120 0 0" rpy="0 ${-camera_pitch * deg} 0" />
+    <parent link="camera" />
+    <child link="camera_mount" />
   </joint>
   <link name="camera_link" />
   <joint name="camera_link_joint" type="fixed">
-    <origin xyz="0.0164 0.0175 0" />
-    <parent link="camera" />
-    <child link="camera_link" />
+    <origin xyz="-0.0164 -0.0175 0" />
+    <parent link="camera_link" />
+    <child link="camera" />
   </joint>
   <!-- Limb Macro -->
@@ -379,5 +379,5 @@
     <!-- Wrist Ball Joint (Floating Joint) -->
     <xacro:if value="${floating_wrist}">
-      <joint name="gripper_joint_${id}" type="floating">
+      <joint name="gripper_joint_${id}" type="fixed">
         <parent link="wrist_${id}" />
         <child link="gripper_${id}" />

Commit message: Refactored launch files

File: robot_description/loris_description/urdf/loris.urdf.xacro (robot description, xacro)
@@ -20,7 +20,7 @@
 -->
 <robot xmlns:xacro="http://www.ros.org/wiki/xacro" name="loris">
-  <!-- Represent wrist as 1 floating joint instead of 3 passive joints -->
-  <xacro:arg name="floating_wrist" default="false" />
-  <xacro:property name="floating_wrist" value="$(arg floating_wrist)" />
+  <!-- Represent wrist as floating joint, fixed joint, or 3 revolute joints -->
+  <xacro:arg name="wrist_joint" default="revolute" />
+  <xacro:property name="wrist_joint" value="$(arg wrist_joint)" />
   <!-- Camera mounting height (m from body origin to pitch axis) -->
   <xacro:arg name="camera_height" default="0.28" />
@@ -244,5 +244,7 @@
   </link>
   <joint name="camera_pitch_joint" type="fixed">
-    <origin xyz="-0.0120 0 0" rpy="0 ${-camera_pitch * deg} 0" />
+    <origin xyz="${-0.0120 * cos(camera_pitch * deg)} 0
+      ${-0.0120 * sin(camera_pitch * deg)}"
+      rpy="0 ${-camera_pitch * deg} 0" />
     <parent link="camera" />
     <child link="camera_mount" />
@@ -281,5 +283,5 @@
       <collision>
         <geometry>
-          <mesh filename="${collision}/shoulder.STL" scale="1 ${reflect} 1" />
+          <mesh filename="${collision}/shoulder.STL" />
         </geometry>
       </collision>
@@ -308,5 +310,5 @@
       <collision>
         <geometry>
-          <mesh filename="${collision}/upper_limb.STL" scale="1 ${reflect} 1" />
+          <mesh filename="${collision}/upper_limb.STL" />
         </geometry>
       </collision>
@@ -335,5 +337,5 @@
       <collision>
         <geometry>
-          <mesh filename="${collision}/lower_limb.STL" scale="1 ${reflect} 1" />
+          <mesh filename="${collision}/lower_limb.STL" />
         </geometry>
       </collision>
@@ -373,10 +375,17 @@
       <collision>
         <geometry>
-          <mesh filename="${collision}/gripper.STL" scale="1 ${reflect} 1" />
+          <mesh filename="${collision}/gripper.STL" />
         </geometry>
       </collision>
     </link>
     <!-- Wrist Ball Joint (Floating Joint) -->
-    <xacro:if value="${floating_wrist}">
+    <xacro:if value="${wrist_joint == 'floating'}">
+      <joint name="gripper_joint_${id}" type="floating">
+        <parent link="wrist_${id}" />
+        <child link="gripper_${id}" />
+      </joint>
+    </xacro:if>
+    <!-- Wrist Ball Joint (Fixed Joint) -->
+    <xacro:if value="${wrist_joint == 'fixed'}">
       <joint name="gripper_joint_${id}" type="fixed">
         <parent link="wrist_${id}" />
@@ -385,6 +394,11 @@
     </xacro:if>
     <!-- Wrist Ball Joint (3-Axis Joint) -->
-    <xacro:unless  value="${floating_wrist}">
-      <link name="wrist_yaw_${id}" />
+    <xacro:if value="${wrist_joint == 'revolute'}">
+      <link name="wrist_yaw_${id}">
+        <inertial>
+          <xacro:inertial mass="0.0001"
+            ixx="0.0000001" iyy="0.0000001" izz="0.0000001" />
+        </inertial>
+      </link>
       <joint name="wrist_yaw_joint_${id}" type="continuous">
         <parent link="wrist_${id}" />
@@ -392,5 +406,10 @@
         <axis xyz="1 0 0" />
       </joint>
-      <link name="wrist_pitch_${id}" />
+      <link name="wrist_pitch_${id}">
+        <inertial>
+          <xacro:inertial mass="0.0001"
+            ixx="0.0000001" iyy="0.0000001" izz="0.0000001" />
+        </inertial>
+      </link>
       <joint name="wrist_pitch_joint_${id}" type="revolute">
         <parent link="wrist_yaw_${id}" />
@@ -407,5 +426,5 @@
           effort="0" velocity="0"/>
       </joint>
-    </xacro:unless>
+    </xacro:if>
   </xacro:macro>
   <!-- Limbs -->
