Commit message: Updated TF structure and integrated IMU

File: climb_control/test/resources/test_robot.urdf (robot description, URDF)
Before this commit: robot test_robot, 10 links, 9 joints
Links:
- removed link root
- added link base_link
Joints:
- removed joint root_joint
- added joint base_joint: type fixed, parent base_link, child body

File: robot_description/loris_description/urdf/loris.urdf.xacro (robot description, xacro)
@@ -86,8 +86,8 @@
       izz="${mass * izz}" />
   </xacro:macro>
-  <!-- Root frame -->
-  <link name="root" />
-  <joint name="root_joint" type="fixed">
-    <parent link="root" />
+  <!-- Base frame -->
+  <link name="base_link" />
+  <joint name="base_joint" type="fixed">
+    <parent link="base_link" />
     <child link="body_front" />
   </joint>
@@ -196,7 +196,7 @@
   </link>
   <joint name="mast_joint" type="fixed">
-    <origin xyz="-0.0247 0 0" />
-    <parent link="mast" />
-    <child link="root" />
+    <origin xyz="0.0247 0 0" />
+    <parent link="body_front" />
+    <child link="mast" />
   </joint>
   <link name="camera_mount">
@@ -220,7 +220,7 @@
   <joint
     name="camera_mast_joint" type="fixed">
-    <origin xyz="0 0 ${-camera_height}" />
-    <parent link="camera_mount" />
-    <child link="mast" />
+    <origin xyz="0 0 ${camera_height}" />
+    <parent link="mast" />
+    <child link="camera_mount" />
   </joint>
   <link
@@ -244,15 +244,13 @@
   </link>
   <joint name="camera_pitch_joint" type="fixed">
-    <origin xyz="${-0.0120 * cos(camera_pitch * deg)} 0
-      ${-0.0120 * sin(camera_pitch * deg)}"
-      rpy="0 ${-camera_pitch * deg} 0" />
-    <parent link="camera" />
-    <child link="camera_mount" />
+    <origin xyz="0.0120 0 0" rpy="0 ${camera_pitch * deg} 0" />
+    <parent link="camera_mount" />
+    <child link="camera" />
   </joint>
   <link name="camera_link" />
   <joint name="camera_link_joint" type="fixed">
-    <origin xyz="-0.0164 -0.0175 0" />
-    <parent link="camera_link" />
-    <child link="camera" />
+    <origin xyz="0.0164 0.0175 0" />
+    <parent link="camera" />
+    <child link="camera_link" />
   </joint>
   <!-- Limb Macro -->

Commit message: Fixed controller test case

File: climb_control/test/resources/test_robot.urdf (robot description, URDF)
Before this commit: robot test_robot, 10 links, 9 joints
Joints:
- joint left_hip: limit lower=-1.57 upper=1.57 effort=1 velocity=1 -> lower=-1.57 upper=1.57 effort=10 velocity=1
- joint left_knee: limit lower=-1.57 upper=1.57 effort=1 velocity=1 -> lower=-1.57 upper=1.57 effort=10 velocity=1
- joint right_hip: limit lower=-1.57 upper=1.57 effort=1 velocity=1 -> lower=-1.57 upper=1.57 effort=10 velocity=1
- joint right_knee: limit lower=-1.57 upper=1.57 effort=1 velocity=1 -> lower=-1.57 upper=1.57 effort=10 velocity=1
